File: pcb/ad9958-dev.kicad_pcb (KiCad board)
At the start: 4 copper layers, 40 x 32 mm, 88 parts, among them J1 INTERFACE, J2 5V, J3 OUT1, J4 OUT0, U1 AZ1117CH-1.8TRG1, U2 AD9958, U3 LMH6714MF, U4 LMH6714MF, X1 25 MHz

Commit message: Gerber export
Parts:
- moved R12 6.26 mm to (179.5, 91.0), turned to 180 degrees
- moved J2 4.92 mm to (180.2, 97.6)
- moved E3 4.42 mm to (183.5, 95.0), turned to 270 degrees
Routing:
- net -5: track 52.8 -> 42.0 mm
- net Net-(E3-Pad1): track 1.80 -> 5.61 mm
- net Net-(E2-Pad2): track 6.87 -> 3.14 mm
- net Net-(E3-Pad2): track 2.09 -> 2.77 mm
